File: snaphat.kicad_pcb (KiCad board)
At the start: 2 copper layers, 100 x 99.4 mm, 133 parts, among them J1 Conn_01x08_S8B-PH-K-S(LF)(SN), J10 P70-6000045R, J11 P70-6000045R, J12 P70-6000045R, J2 Conn_02x20_2214SM-40G-75-PCR, J3 Conn_01x02_B2B-PH-K-S(LF)(SN), J4 USB_C_USB4930-00-A, J5 Conn_01x03_MC34747, J6 Conn_01x04_FFC3B11-04-T, J7 Conn_01x04_FFC3B11-04-T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

Commit message: Update README and docs
Other:
- board text added: "Prepared for manufacturing at JLCPCB - Standard PCB - 2 layers - min. via hole size/diameter: 0.3/0.4mm"
- board text removed: "Prepared for manufacturing at JLCPCB - Standard PCB - min. via hole size/diameter: 0.3/0.4mm"
Changed lines of the file:
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@@
 		(allow_soldermask_bridges_in_footprints no)
 		(tenting front back)
+		(aux_axis_origin 146.64 159.819)
 		(grid_origin 169.25 131.679)
 		(pcbplotparams
@@
 			)
 			(rotate
-				(xyz -90 -0 -0)
+				(xyz -90 0 0)
 			)
 		)
@@
 			)
 			(rotate
-				(xyz -90 -0 -0)
+				(xyz -90 0 0)
 			)
 		)
@@
 			)
 			(rotate
-				(xyz -90 -0 -0)
+				(xyz -90 0 0)
 			)
 		)
@@
 			)
 			(rotate
-				(xyz -0 -0 -0)
+				(xyz 0 0 0)
 			)
 		)
@@
 			)
 			(rotate
-				(xyz -90 -0 -0)
+				(xyz -90 0 0)
 			)
 		)
@@
 			)
 			(rotate
-				(xyz -0 -0 -0)
+				(xyz 0 0 0)
 			)
 		)
@@
 			)
 			(rotate
-				(xyz -0 -0 -0)
+				(xyz 0 0 0)
 			)
 		)
@@
 			)
 			(rotate
-				(xyz -90 -0 -0)
+				(xyz -90 0 0)
 			)
 		)
@@
 			)
 			(rotate
-				(xyz -0 -0 -0)
+				(xyz 0 0 0)
 			)
 		)
@@
 			)
 			(rotate
-				(xyz -90 -0 -0)
+				(xyz -90 0 0)
 			)
 		)
@@
 			)
 			(rotate
-				(xyz -0 -0 -0)
+				(xyz 0 0 0)
 			)
 		)
@@
 			)
 			(rotate
-				(xyz -90 -0 -0)
+				(xyz -90 0 0)
 			)
 		)
@@
 			)
 			(rotate
-				(xyz -90 -0 -0)
+				(xyz -90 0 0)
 			)
 		)
@@
 			)
 			(rotate
-				(xyz -0 -0 -0)
+				(xyz 0 0 0)
 			)
 		)
@@
 			)
 			(rotate
-				(xyz -90 -0 -0)
+				(xyz -90 0 0)
 			)
 		)
@@
 			)
 			(rotate
-				(xyz -90 -0 -180)
+				(xyz -90 0 -180)
 			)
 		)
@@
 			)
 			(rotate
-				(xyz -0 -0 -0)
+				(xyz 0 0 0)
 			)
 		)
@@
 			)
 			(rotate
-				(xyz -90 -0 -0)
+				(xyz -90 0 0)
 			)
 		)
@@
 			)
 			(rotate
-				(xyz -90 -0 -0)
+				(xyz -90 0 0)
 			)
 		)
@@
 			)
 			(rotate
-				(xyz -90 -0 -0)
+				(xyz -90 0 0)
 			)
 		)
@@
 			)
 			(rotate
-				(xyz -0 -0 -0)
+				(xyz 0 0 0)
 			)
 		)
@@
 			)
 			(rotate
-				(xyz -90 -0 -0)
+				(xyz -90 0 0)
 			)
 		)
@@
 			)
 			(rotate
-				(xyz -90 -0 -0)
+				(xyz -90 0 0)
 			)
 		)
@@
 			)
 			(rotate
-				(xyz -90 -0 90)
+				(xyz -90 0 90)
 			)
 		)
@@
 			)
 			(rotate
-				(xyz -90 -0 -0)
+				(xyz -90 0 0)
 			)
 		)
@@
 			)
 			(rotate
-				(xyz -90 -0 -0)
+				(xyz -90 0 0)
 			)
 		)
@@
 			)
 			(rotate
-				(xyz -90 -0 -0)
+				(xyz -90 0 0)
 			)
 		)
@@
 			)
 			(rotate
-				(xyz -90 -0 -0)
+				(xyz -90 0 0)
 			)
 		)
@@
 			)
 			(rotate
-				(xyz -90 -0 -0)
+				(xyz -90 0 0)
 			)
 		)
@@
 			)
 			(rotate
-				(xyz -90 -0 -0)
+				(xyz -90 0 0)
 			)
 		)
@@
 			)
 			(rotate
-				(xyz 180 -0 -0)
+				(xyz 180 0 0)
 			)
 		)
@@
 			)
 			(rotate
-				(xyz -90 -0 -0)
+				(xyz -90 0 0)
 			)
 		)
@@
 			)
 			(rotate
-				(xyz 90 -0 90)
+				(xyz 90 0 90)
 			)
 		)
@@
 			)
 			(rotate
-				(xyz -0 180 90)
+				(xyz 0 180 90)
 			)
 		)
@@
 			)
 			(rotate
-				(xyz -0 -0 -0)
+				(xyz 0 0 0)
 			)
 		)
@@
 			)
 			(rotate
-				(xyz -90 -0 -0)
+				(xyz -90 0 0)
 			)
 		)
@@
 			)
 			(rotate
-				(xyz -0 -0 -90)
+				(xyz 0 0 -90)
 			)
 		)
@@
 			)
 			(rotate
-				(xyz -90 -0 -180)
+				(xyz -90 0 -180)
 			)
 		)
@@
 			)
 			(rotate
-				(xyz -90 -0 -180)
+				(xyz -90 0 -180)
 			)
 		)
@@
 			)
 			(rotate
-				(xyz -90 -0 -0)
+				(xyz -90 0 0)
 			)
 		)
@@
 			)
 			(rotate
-				(xyz -90 -0 -0)
+				(xyz -90 0 0)
 			)
 		)
@@
 	)
 	(gr_text "VBAT"
-		(at 239.19 111.01 -0)
+		(at 239.19 111.01 0)
 		(layer "B.SilkS")
 		(effects
@@
 	)
 	(gr_text "GND"
-		(at 153.974977 77.400173 -0)
+		(at 153.974977 77.400173 0)
 		(layer "B.SilkS")
 		(effects
@@
 		)
 	)
-	(gr_text "Prepared for manufacturing at JLCPCB\n	- Standard PCB\n	- min. via hole size/diameter: 0.3/0.4mm"
+	(gr_text "Prepared for manufacturing at JLCPCB\n	- Standard PCB\n	- 2 layers\n	- min. via hole size/diameter: 0.3/0.4mm"
 		(at 158.9 157.85 0)
 		(layer "Cmts.User")
@@
 		)
 	)
+	(dimension
+		(type orthogonal)
+		(layer "Cmts.User")
+		(pts
+			(xy 208.7 129.699) (xy 208.2 159.819)
+		)
+		(height 7.85)
+		(orientation 1)
+		(format
+			(prefix "")
+			(suffix "")
+			(units 3)
+			(units_format 0)
+			(precision 2)
+			(suppress_zeroes yes)
+		)
+		(style
+			(thickness 0.1)
+			(arrow_length 1.27)
+			(text_position_mode 0)
+			(arrow_direction outward)
+			(extension_height 0.58642)
+			(extension_offset 0.5)
+			(keep_text_aligned yes)
+		)
+		(gr_text "30.12"
+			(at 215.4 144.759 90)
+			(layer "Cmts.User")
+			(effects
+				(font
+					(size 1 1)
+					(thickness 0.15)
+				)
+			)
+		)
+	)
+	(dimension
+		(type orthogonal)
+		(layer "Cmts.User")
+		(pts
+			(xy 243.649954 128.5) (xy 243.649999 60.401321)
+		)
+		(height 7.940046)
+		(orientation 1)
+		(format
+			(prefix "")
+			(suffix "")
+			(units 3)
+			(units_format 0)
+			(precision 2)
+			(suppress_zeroes yes)
+		)
+		(style
+			(thickness 0.1)
+			(arrow_length 1.27)
+			(text_position_mode 0)
+			(arrow_direction outward)
+			(extension_height 0.58642)
+			(extension_offset 0.5)
+			(keep_text_aligned yes)
+		)
+		(gr_text "68.1"
+			(at 250.44 94.45066 90)
+			(layer "Cmts.User")
+			(effects
+				(font
+					(size 1 1)
+					(thickness 0.15)
+				)
+			)
+		)
+	)
+	(dimension
+		(type orthogonal)
+		(layer "Cmts.User")
+		(pts
+			(xy 146.64 156.759) (xy 211.76 156.759)
+		)
+		(height 6.2)
+		(orientation 0)
+		(format
+			(prefix "")
+			(suffix "")
+			(units 3)
+			(units_format 0)
+			(precision 2)
+			(suppress_zeroes yes)
+		)
+		(style
+			(thickness 0.1)
+			(arrow_length 1.27)
+			(text_position_mode 0)
+			(arrow_direction outward)
+			(extension_height 0.58642)
+			(extension_offset 0.5)
+			(keep_text_aligned yes)
+		)
+		(gr_text "65.12"
+			(at 179.2 161.809 0)
+			(layer "Cmts.User")
+			(effects
+				(font
+					(size 1 1)
+					(thickness 0.15)
+				)
+			)
+		)
+	)
+	(dimension
+		(type orthogonal)
+		(layer "Cmts.User")
+		(pts
+			(xy 246.6513 63.401363) (xy 146.65 63.399)
+		)
+		(height -6.782363)
+		(orientation 0)
+		(format
+			(prefix "")
+			(suffix "")
+			(units 3)
+			(units_format 0)
+			(precision 2)
+			(suppress_zeroes yes)
+		)
+		(style
+			(thickness 0.1)
+			(arrow_length 1.27)
+			(text_position_mode 0)
+			(arrow_direction outward)
+			(extension_height 0.58642)
+			(extension_offset 0.5)
+			(keep_text_aligned yes)
+		)
+		(gr_text "100"
+			(at 196.65065 55.469 0)
+			(layer "Cmts.User")
+			(effects
+				(font
+					(size 1 1)
+					(thickness 0.15)
+				)
+			)
+		)
+	)
