File: snaphat.kicad_sch (KiCad schematic)
At the start: 105 parts, among them J1 Conn_01x08_S8B-PH-K-S(LF)(SN), J10 P70-6000045R, J11 P70-6000045R, J12 P70-6000045R, J2 Conn_02x20_2214SM-40G-75-PCR, J3 Conn_01x02_B2B-PH-K-S(LF)(SN), J4 USB_C_USB4930-00-A, J5 Conn_01x03_MC34747, J6 Conn_01x04_SFV4R-3STBE1HLF/C, J7 Conn_01x04_SFV4R-3STBE1HLF/C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

Commit message: Add FFC cable info
Parts:
- added H57: 05-04-D-0050-A-4-06-4-T, symbol library:05-04-D-0050-A-4-06-4-T
Other:
- note added: "FFC cable:"
Changed lines of the file:
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@@
 		)
 	)
+	(text "FFC cable:"
+		(exclude_from_sim no)
+		(at 323.596 115.316 0)
+		(effects
+			(font
+				(face "Quicksand")
+				(size 1.27 1.27)
+				(thickness 0.1588)
+			)
+			(justify left bottom)
+		)
+	)
 	(text "GPIO8(CE0)"
 		(exclude_from_sim no)
@@
 		)
 		(property "Value" "5k1"
-			(at 218.44 66.04 90)
+			(at 217.932 66.04 90)
 			(effects
 				(font
@@
 					(unit 1)
 				)
+			)
+		)
+	)
+	(symbol
+		(lib_id "library:05-04-D-0050-A-4-06-4-T")
+		(at 327.66 116.84 0)
+		(unit 1)
+		(exclude_from_sim no)
+		(in_bom yes)
+		(on_board yes)
+		(dnp no)
+		(property "Reference" "H57"
+			(at 323.342 118.11 0)
+			(effects
+				(font
+					(size 1.27 1.27)
+				)
+				(justify left)
+			)
+		)
+		(property "Value" "05-04-D-0050-A-4-06-4-T"
+			(at 335.026 118.11 0)
+			(effects
+				(font
+					(size 1.27 1.27)
+				)
+				(justify left)
+			)
+		)
+		(property "Footprint" ""
+			(at 327.66 116.84 0)
+			(effects
+				(font
+					(size 1.27 1.27)
+				)
+				(hide yes)
+			)
+		)
+		(property "Datasheet" ""
+			(at 327.66 116.84 0)
+			(effects
+				(font
+					(size 1.27 1.27)
+				)
+				(hide yes)
+			)
+		)
+		(property "Description" "FFC / FPC Cable, 4 Core, 0.5 mm, Opposite Sided Contacts, 1.97 \", 50 mm, White"
+			(at 327.66 116.84 0)
+			(effects
+				(font
+					(size 1.27 1.27)
+				)
+				(hide yes)
+			)
+		)
+		(property "Part number" "05-04-D-0050-A-4-06-4-T"
+			(at 327.66 116.84 0)
+			(effects
+				(font
+					(size 1.27 1.27)
+				)
+				(hide yes)
+			)
+		)
+		(property "Manufacturer" "GCT"
+			(at 332.74 118.11 0)
+			(effects
+				(font
+					(size 1.27 1.27)
+				)
+			)
+		)
+		(property "Category" "OTS"
+			(at 327.66 116.84 0)
+			(effects
+				(font
+					(size 1.27 1.27)
+				)
+				(hide yes)
+			)
+		)
+		(instances
+			(project ""
+				(path "/1b9269fa-3ac8-429a-ab83-4cc9a4203d51"
+					(reference "H57")
+					(unit 1)
+				)

Commit message: Fixes to library, add updated schematic PDF and BOM
Parts:
- D7: Manufacturer (none) -> Vishay; Part number (none) -> SL04-E3-08
- D9: Manufacturer LITTELFUSE -> Littelfuse
- H19, H20, H21, H22, H23, H24, H25, H52: Category Double ended 150mm crimp contact wire -> Wire harness
- H57: Category OTS -> Wire harness
Changed lines of the file:
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@@
 			)
 		)
-		(property "Manufacturer" "LITTELFUSE"
+		(property "Manufacturer" "Littelfuse"
 			(at -282.83 110.49 0)
 			(effects
@@
 			)
 		)
+		(property "Part number" "SL04-E3-08"
+			(at 233.68 60.96 0)
+			(effects
+				(font
+					(size 1.27 1.27)
+				)
+				(hide yes)
+			)
+		)
+		(property "Manufacturer" "Vishay"
+			(at 233.68 60.96 0)
+			(effects
+				(font
+					(size 1.27 1.27)
+				)
+				(hide yes)
+			)
+		)
 		(pin "1"
 		)
@@
 			)
 		)
-		(property "Description" "Miscellaneous component"
+		(property "Description" "Double ended 150mm crimp contact wire"
 			(at 22.86 63.5 0)
 			(effects
@@
 			)
 		)
-		(property "Category" "Double ended 150mm crimp contact wire"
+		(property "Category" "Wire harness"
 			(at 22.86 63.5 0)
 			(effects
@@
 			)
 		)
-		(property "Description" "Miscellaneous component"
+		(property "Description" "Double ended 150mm crimp contact wire"
 			(at 22.86 78.74 0)
 			(effects
@@
 			)
 		)
-		(property "Category" "Double ended 150mm crimp contact wire"
+		(property "Category" "Wire harness"
 			(at 22.86 78.74 0)
 			(effects
@@
 			)
 		)
-		(property "Description" "Miscellaneous component"
+		(property "Description" "Double ended 150mm crimp contact wire"
 			(at 22.86 59.69 0)
 			(effects
@@
 			)
 		)
-		(property "Category" "Double ended 150mm crimp contact wire"
+		(property "Category" "Wire harness"
 			(at 22.86 59.69 0)
 			(effects
@@
 			)
 		)
-		(property "Description" "Miscellaneous component"
+		(property "Description" "Double ended 150mm crimp contact wire"
 			(at 22.86 74.93 0)
 			(effects
@@
 			)
 		)
-		(property "Category" "Double ended 150mm crimp contact wire"
+		(property "Category" "Wire harness"
 			(at 22.86 74.93 0)
 			(effects
@@
 			)
 		)
-		(property "Description" "Miscellaneous component"
+		(property "Description" "Double ended 150mm crimp contact wire"
 			(at 22.86 67.31 0)
 			(effects
@@
 			)
 		)
-		(property "Category" "Double ended 150mm crimp contact wire"
+		(property "Category" "Wire harness"
 			(at 22.86 67.31 0)
 			(effects
@@
 			)
 		)
-		(property "Description" "Miscellaneous component"
+		(property "Description" "Double ended 150mm crimp contact wire"
 			(at 22.86 71.12 0)
 			(effects
@@
 			)
 		)
-		(property "Category" "Double ended 150mm crimp contact wire"
+		(property "Category" "Wire harness"
 			(at 22.86 71.12 0)
 			(effects
@@
 			)
 		)
-		(property "Description" "Miscellaneous component"
+		(property "Description" "Double ended 150mm crimp contact wire"
 			(at 22.86 55.88 0)
 			(effects
@@
 			)
 		)
-		(property "Category" "Double ended 150mm crimp contact wire"
+		(property "Category" "Wire harness"
 			(at 22.86 55.88 0)
 			(effects
@@
 			)
 		)
-		(property "Category" "OTS"
+		(property "Category" "Wire harness"
 			(at 327.66 116.84 0)
 			(effects
@@
 			)
 		)
-		(property "Description" "Miscellaneous component"
+		(property "Description" "Double ended 150mm crimp contact wire"
 			(at 22.86 52.07 0)
 			(effects
@@
 			)
 		)
-		(property "Category" "Double ended 150mm crimp contact wire"
+		(property "Category" "Wire harness"
 			(at 22.86 52.07 0)
 			(effects

Commit message: Add LED_SHUTTER
Connections:
- net LED_SHUTTER: now reaches J2.36 (Pin_36)
- net LOW_BATTERY renamed LED_LBO
- no-connect marks 8 -> 7
Other:
- sheet Power supply renamed Power supply and LEDs
- sheet Power supply and LEDs ports: added LED_LBO, LED_SHUTTER; removed LOW_BATTERY
- moved on the sheet: H33, H38, H39, H51, J3

Commit message: Replace FFC connector with 1mm pitch
Parts:
- H57: value 05-04-D-0050-A-4-06-4-T -> 10-04-D-0030-C-4-08-4-T; symbol library:05-04-D-0050-A-4-06-4-T -> library:10-04-D-0030-C-4-08-4-T; Part number 05-04-D-0050-A-4-06-4-T -> 10-04-D-0030-C-4-08-4-T
- J6, J7: value Conn_01x04_SFV4R-3STBE1HLF/C -> Conn_01x04_FFC3B11-04-T; footprint library:AMPHENOL_SFV4R-3STBE1HLF -> library:GCT_FFC3B11-04-T; symbol library:Conn_01x04_SFV4R-3STBE1HLF/C -> library:Conn_01x04_FFC3B11-04-T; Manufacturer Amphenol -> GCT; Part number SFV4R-3STBE1HLF/C -> FFC3B11-04-T
Connections:
- net GND: now also J6.4 (Pin_4); no longer J6.1 (Pin_1)
- net GND_EXT: now also J7.4 (Pin_4); no longer J7.1 (Pin_1)
- net Power supply and LEDs/VBUS: now also J6.1 (Pin_1); no longer J6.4 (Pin_4)
- net USBC_DATA_N: now also J6.2 (Pin_2); no longer J6.3 (Pin_3)
- net USBC_DATA_P: now also J6.3 (Pin_3); no longer J6.2 (Pin_2)
- net USBC_EXT_DATA_N: now also J7.2 (Pin_2); no longer J7.3 (Pin_3)
- net USBC_EXT_DATA_P: now also J7.3 (Pin_3); no longer J7.2 (Pin_2)
- net VBUS_EXT: now also J7.1 (Pin_1); no longer J7.4 (Pin_4)
Other:
- moved on the sheet: J7
Changed lines of the file:
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@@
 	)
 	(symbol
-		(lib_id "library:Conn_01x04_SFV4R-3STBE1HLF/C")
-		(at 262.89 78.74 0)
-		(mirror x)
+		(lib_id "library:Conn_01x04_FFC3B11-04-T")
+		(at 262.89 76.2 0)
 		(unit 1)
 		(exclude_from_sim no)
@@
 		(dnp no)
 		(property "Reference" "J6"
-			(at 262.89 84.074 0)
+			(at 262.89 70.612 0)
 			(effects
 				(font
@@
 			)
 		)
-		(property "Value" "Conn_01x04_SFV4R-3STBE1HLF/C"
-			(at 262.89 85.09 0)
+		(property "Value" "Conn_01x04_FFC3B11-04-T"
+			(at 265.938 75.438 90)
 			(effects
 				(font
-					(face "Quicksand")
 					(size 1.27 1.27)
 				)
@@
 			)
 		)
-		(property "Footprint" "library:AMPHENOL_SFV4R-3STBE1HLF"
-			(at 262.89 78.74 0)
+		(property "Footprint" "library:GCT_FFC3B11-04-T"
+			(at 262.89 76.2 0)
 			(effects
 				(font
-					(face "Quicksand")
 					(size 1.27 1.27)
 				)
@@
 		)
 		(property "Datasheet" "~"
-			(at 262.89 78.74 0)
+			(at 262.89 76.2 0)
 			(effects
 				(font
-					(face "Quicksand")
 					(size 1.27 1.27)
 				)
@@
 			)
 		)
-		(property "Description" "Generic connector, single row, 01x04, script generated (kicad-library-utils/schlib/autogen/connector/)"
-			(at 262.89 78.74 0)
+		(property "Description" "4 Position FFC, FPC Connector Contacts, Top 0.039\" (1.00mm) Surface Mount, Right Angle"
+			(at 262.89 76.2 0)
 			(effects
 				(font
-					(face "Quicksand")
 					(size 1.27 1.27)
 				)
@@
 			)
 		)
-		(property "Part number" "SFV4R-3STBE1HLF/C"
-			(at 265.684 76.962 90)
+		(property "Part number" "FFC3B11-04-T"
+			(at 265.684 77.216 90)
 			(effects
 				(font
-					(face "Quicksand")
 					(size 1.27 1.27)
 				)
 			)
 		)
-		(property "Manufacturer" "Amphenol"
-			(at 262.89 78.74 0)
+		(property "Manufacturer" "GCT"
+			(at 262.89 76.2 0)
 			(effects
 				(font
-					(face "Quicksand")
 					(size 1.27 1.27)
 				)
@@
 	)
 	(symbol
-		(lib_id "library:Conn_01x04_SFV4R-3STBE1HLF/C")
-		(at 341.63 62.23 180)
+		(lib_id "library:Conn_01x04_FFC3B11-04-T")
+		(at 341.63 59.69 0)
+		(mirror y)
 		(unit 1)
 		(exclude_from_sim no)
@@
 		(dnp no)
 		(property "Reference" "J7"
-			(at 341.63 67.564 0)
+			(at 341.63 54.102 0)
 			(effects
 				(font
@@
 			)
 		)
-		(property "Value" "Conn_01x04_SFV4R-3STBE1HLF/C"
-			(at 341.63 68.58 0)
+		(property "Value" "Conn_01x04_FFC3B11-04-T"
+			(at 341.63 67.31 0)
 			(effects
 				(font
-					(face "Quicksand")
 					(size 1.27 1.27)
 				)
@@
 			)
 		)
-		(property "Footprint" "library:AMPHENOL_SFV4R-3STBE1HLF"
-			(at 341.63 62.23 0)
+		(property "Footprint" "library:GCT_FFC3B11-04-T"
+			(at 341.63 59.69 0)
 			(effects
 				(font
-					(face "Quicksand")
 					(size 1.27 1.27)
 				)
@@
 		)
 		(property "Datasheet" "~"
-			(at 341.63 62.23 0)
+			(at 341.63 59.69 0)
 			(effects
 				(font
-					(face "Quicksand")
 					(size 1.27 1.27)
 				)
@@
 			)
 		)
-		(property "Description" "Generic connector, single row, 01x04, script generated (kicad-library-utils/schlib/autogen/connector/)"
-			(at 341.63 62.23 0)
+		(property "Description" "4 Position FFC, FPC Connector Contacts, Top 0.039\" (1.00mm) Surface Mount, Right Angle"
+			(at 341.63 59.69 0)
 			(effects
 				(font
-					(face "Quicksand")
 					(size 1.27 1.27)
 				)
@@
 			)
 		)
-		(property "Part number" "SFV4R-3STBE1HLF/C"
-			(at 338.836 60.706 90)
+		(property "Part number" "FFC3B11-04-T"
+			(at 339.09 60.452 90)
 			(effects
 				(font
-					(face "Quicksand")
 					(size 1.27 1.27)
 				)
 			)
 		)
-		(property "Manufacturer" "Amphenol"
-			(at 341.63 62.23 0)
+		(property "Manufacturer" "GCT"
+			(at 341.63 59.69 0)
 			(effects
 				(font
-					(face "Quicksand")
 					(size 1.27 1.27)
 				)
@@
 	)
 	(symbol
-		(lib_id "library:05-04-D-0050-A-4-06-4-T")
+		(lib_id "library:10-04-D-0030-C-4-08-4-T ")
 		(at 327.66 116.84 0)
 		(unit 1)
@@
 			)
 		)
-		(property "Value" "05-04-D-0050-A-4-06-4-T"
-			(at 335.026 118.11 0)
+		(property "Value" "10-04-D-0030-C-4-08-4-T"
+			(at 331.724 119.634 0)
 			(effects
 				(font
@@
 			)
 		)
-		(property "Description" "FFC / FPC Cable, 4 Core, 0.5 mm, Opposite Sided Contacts, 1.97 \", 50 mm, White"
+		(property "Description" "FFC / FPC Cable, 4 Core, 1 mm, Opposite Sided Contacts, 30 mm, White"
 			(at 327.66 116.84 0)
 			(effects
@@
 			)
 		)
-		(property "Part number" "05-04-D-0050-A-4-06-4-T"
+		(property "Part number" "10-04-D-0030-C-4-08-4-T"
 			(at 327.66 116.84 0)
 			(effects
@@
 		)
 		(property "Manufacturer" "GCT"
-			(at 332.74 118.11 0)
+			(at 332.486 118.11 0)
 			(effects
 				(font

Commit message: Reroute USB, add shutter LED signal pulldown
Changed lines of the file:
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@@
 			(effects
 				(font
+					(face "Quicksand")
 					(size 1.27 1.27)
 				)
@@
 			(effects
 				(font
+					(face "Quicksand")
 					(size 1.27 1.27)
 				)
@@
 			(effects
 				(font
+					(face "Quicksand")
 					(size 1.27 1.27)
 				)
@@
 			(effects
 				(font
+					(face "Quicksand")
 					(size 1.27 1.27)
 				)
@@
 			(effects
 				(font
+					(face "Quicksand")
 					(size 1.27 1.27)
 				)
@@
 			(effects
 				(font
+					(face "Quicksand")
 					(size 1.27 1.27)
 				)
@@
 			(effects
 				(font
+					(face "Quicksand")
 					(size 1.27 1.27)
 				)
@@
 			(effects
 				(font
+					(face "Quicksand")
 					(size 1.27 1.27)
 				)
@@
 			(effects
 				(font
+					(face "Quicksand")
 					(size 1.27 1.27)
 				)
@@
 			(effects
 				(font
+					(face "Quicksand")
 					(size 1.27 1.27)
 				)
@@
 			(effects
 				(font
+					(face "Quicksand")
 					(size 1.27 1.27)
 				)
@@
 			(effects
 				(font
+					(face "Quicksand")
 					(size 1.27 1.27)
 				)
@@
 			(effects
 				(font
+					(face "Quicksand")
 					(size 1.27 1.27)
 				)
@@
 			(effects
 				(font
+					(face "Quicksand")
 					(size 1.27 1.27)
 				)
@@
 			(effects
 				(font
+					(face "Quicksand")
 					(size 1.27 1.27)
 				)
@@
 		)
 		(property "Value" "10-04-D-0030-C-4-08-4-T"
-			(at 331.724 119.634 0)
+			(at 335.28 118.11 0)
 			(effects
 				(font
+					(face "Quicksand")
 					(size 1.27 1.27)
 				)
@@
 			(effects
 				(font
+					(face "Quicksand")
 					(size 1.27 1.27)
 				)
@@
 			(effects
 				(font
+					(face "Quicksand")
 					(size 1.27 1.27)
 				)
@@
 			(effects
 				(font
+					(face "Quicksand")
 					(size 1.27 1.27)
 				)
@@
 			(effects
 				(font
+					(face "Quicksand")
 					(size 1.27 1.27)
 				)
@@
 			(effects
 				(font
+					(face "Quicksand")
 					(size 1.27 1.27)
 				)
@@
 			(effects
 				(font
+					(face "Quicksand")
 					(size 1.27 1.27)
 				)
