File: usb_hat/usb_hat.kicad_sch (KiCad schematic)
At the start: 15 parts, among them J1 Conn_01x04_FFC3B11-04-T, J2 P70-6000045R, J3 P70-6000045R, J4 P70-6000045R, J5 P70-6000045R, J6 P70-6000045R

Commit message: Fix P70-6000045R missing from BOM
Parts:
- J2, J3, J4, J5, J6: Manufacturer (none) -> Harwin; Part number (none) -> P70-6000045R; now in the parts list
